Commit message: yeni gazebo için launcherlar uyarlandı. urdfte ufak düzenlemeler yapıldı.

File: src/kasva_description/urdf/camera.xacro (robot description, xacro)
@@ -20,8 +20,8 @@
         />
     </link>
-    <joint name="base_camera_joint" type="fixed">
-        <parent link="base_link"/>
+    <joint name="chasis_camera_joint" type="fixed">
+        <parent link="chasis"/>
         <child link="camera_link"/>
-        <origin xyz="${base_l_x / 2.0} 0 ${base_l_z / 2.0 - camera_l_z}" rpy="0 0 0"/>
+        <origin xyz="${chasis_l_x / 2.0} 0 ${chasis_l_z / 2.0 - camera_l_z}" rpy="0 0 0"/>
     </joint>
     <!-- opencv ile çalışmak için kameranın x ekseni, z ekseni olması lazım çünkü görüntüyü öyle tasavvur ediyor -->

File: src/kasva_description/urdf/display.urdf.xacro (robot description, xacro)
@@ -5,5 +5,5 @@
     <xacro:include filename="links.xacro"/>
     <xacro:include filename="joints.xacro"/>
-    <!-- <xacro:include filename="lidar.xacro"/> -->
-    <!-- <xacro:include filename="camera.xacro"/> -->
+    <xacro:include filename="lidar.xacro"/>
+    <xacro:include filename="camera.xacro"/>
 </robot>

File: src/kasva_description/urdf/g_plugins.xacro (robot description, xacro)
@@ -1,45 +1,96 @@
 <?xml version="1.0"?>
 <robot xmlns:xacro="http://www.ros.org/wiki/xacro">
-    <!-- LIDAR Plugin (Örnek Fortress için uyarlanmış bir lidar plugin'i) -->
+    <!-- Reference -->
     <gazebo reference="laser_frame">
-        <material>Gazebo/Black</material>
-        <sensor name="laser" type="ray">
+        <sensor name='gpu_lidar' type='gpu_lidar'>"
+            <lidar>
+                <scan>
+                    <horizontal>
+                        <samples>640</samples>
+                        <resolution>1</resolution>
+                        <min_angle>-1.396263</min_angle>
+                        <max_angle>1.396263</max_angle>
+                    </horizontal>
+                    <vertical>
+                        <samples>1</samples>
+                        <resolution>0.01</resolution>
+                        <min_angle>0</min_angle>
+                        <max_angle>0</max_angle>
+                    </vertical>
+                </scan>
+                <range>
+                    <min>0.08</min>
+                    <max>10.0</max>
+                    <resolution>0.01</resolution>
+                </range>
+            </lidar>
+            <topic>scan</topic>
+            <update_rate>10</update_rate>
+            <always_on>1</always_on>
+            <visualize>true</visualize>
+            <gz_frame_id>laser_frame</gz_frame_id>
+        </sensor>
+    </gazebo>
+    <gazebo reference="camera_link">
+        <sensor name='camera' type='camera'>
             <pose>0 0 0 0 0 0</pose>
             <visualize>true</visualize>
-            <update_rate>10</update_rate>
-            <ray>
-                <scan>
-                    <horizontal>
-                        <samples>360</samples>
-                        <min_angle>-1.57</min_angle>
-                        <max_angle>1.57</max_angle>
-                    </horizontal>
-                </scan>
-                <range>
-                    <min>0.3</min>
-                    <max>12</max>
-                </range>
-            </ray>
-            <plugin name="ignition_ros_ray_sensor" filename="ignition-gazebo-ray-system">
-                <output_type>sensor_msgs/LaserScan</output_type>
-                <frame_name>laser_frame</frame_name>
-            </plugin>
+            <update_rate>30</update_rate>
+            <camera>
+                <camera_info_topic>camera/camera_info</camera_info_topic>
+                <horizontal_fov>1.089</horizontal_fov>
+                <image>
+                    <format>R8G8B8</format>
+                    <width>640</width>
+                    <height>480</height>
+                </image>
+                <clip>
+                    <near>0.05</near>
+                    <far>8.0</far>
+                </clip>
+            </camera>
+            <topic>camera/image_raw</topic>
+            <gz_frame_id>camera_optical_link</gz_frame_id>
         </sensor>
     </gazebo>
-    <!-- Diff Drive Plugin Fortress için uyarlanmış diff drive sistemi -->
+    <!-- Diff Drive Plugin (Fortress için uyarlanmış) -->
     <gazebo>
-        <plugin filename="ignition-gazebo-diff-drive-system" name="ignition::gazebo::systems::DiffDrive">
-            <!-- Tekerlek eklemleri -->
+        <plugin
+            filename="libignition-gazebo-diff-drive-system.so"
+            name="ignition::gazebo::systems::DiffDrive">
             <left_joint>base_TO_left_wheel</left_joint>
             <right_joint>base_TO_right_wheel</right_joint>
-            <!-- Kinematik parametreler -->
-            <wheel_separation>0.45</wheel_separation>
-            <!-- Eski yapılandırmada wheel_diameter 0.2 idi, bu durumda yarıçap 0.1 m -->
-            <wheel_radius>0.1</wheel_radius>
-            <!-- Odometri ve tf ayarları -->
-            <odom_publish_frequency>20</odom_publish_frequency>
-            <frame_id>odom</frame_id>
-            <child_frame_id>base_link</child_frame_id>
+            <wheel_separation>1.2</wheel_separation>
+            <wheel_radius>0.4</wheel_radius>
+            <odom_publish_frequency>1</odom_publish_frequency>
+            <topic>cmd_vel</topic>
         </plugin>
+        <plugin filename="libignition-gazebo6-joint-state-publisher-system.so" name="ignition::gazebo::systems::JointStatePublisher">
+            <!-- Yayınlama frekansı (Hz) -->
+            <update_rate>50</update_rate>
+            <!-- Yayınlanacak eklemlerin listesi -->
+            <joint_names>
+                <joint>base_TO_left_wheel</joint>
+                <joint>base_TO_right_wheel</joint>
+                <!-- Diğer eklemleri de ekleyebilirsiniz -->
+            </joint_names>
+        </plugin>
+        <plugin
+            filename="gz-sim-sensors-system"
+            name="gz::sim::systems::Sensors">
+            <render_engine>ogre2</render_engine>
+        </plugin>
+        <!-- ROS Kamera Plugin -->
+        <gazebo>
+            <plugin filename="libgazebo_ros_camera.so" name="ros_camera">
+                <ros>
+                    <namespace>/</namespace>
+                </ros>
+                <camera_name>camera</camera_name>
+                <frame_name>camera_optical_link</frame_name>
+                <hack_baseline>0.07</hack_baseline>
+                <update_rate>10</update_rate>
+            </plugin>
+        </gazebo>
     </gazebo>
 </robot>

File: src/kasva_description/urdf/gazebo.urdf.xacro (robot description, xacro)
@@ -6,4 +6,5 @@
     <xacro:include filename="joints.xacro"/>
     <xacro:include filename="lidar.xacro"/>
+    <xacro:include filename="camera.xacro"/>
     <xacro:include filename="g_plugins.xacro"/>
 </robot>

Commit message: şerit takip için simulasyon ayarlamaları yapıldı. kamera açısı değiştirildi.

File: src/kasva_description/urdf/camera.xacro (robot description, xacro)
@@ -23,5 +23,5 @@
         <parent link="chasis"/>
         <child link="camera_link"/>
-        <origin xyz="${chasis_l_x / 2.0} 0 ${chasis_l_z / 2.0 - camera_l_z}" rpy="0 0 0"/>
+        <origin xyz="${chasis_l_x / 2.0} 0 ${chasis_l_z / 2.0 - camera_l_z}" rpy="0 ${pi/4} 0"/>
     </joint>
     <!-- opencv ile çalışmak için kameranın x ekseni, z ekseni olması lazım çünkü görüntüyü öyle tasavvur ediyor -->

File: src/kasva_description/urdf/g_plugins.xacro (robot description, xacro)
@@ -7,8 +7,8 @@
                 <scan>
                     <horizontal>
-                        <samples>640</samples>
+                        <samples>360</samples>
                         <resolution>1</resolution>
-                        <min_angle>-1.396263</min_angle>
-                        <max_angle>1.396263</max_angle>
+                        <min_angle>-3.141592</min_angle>
+                        <max_angle>3.141592</max_angle>
                     </horizontal>
                     <vertical>
@@ -26,5 +26,5 @@
             </lidar>
             <topic>scan</topic>
-            <update_rate>10</update_rate>
+            <update_rate>5</update_rate>
             <always_on>1</always_on>
             <visualize>true</visualize>
@@ -54,5 +54,4 @@
         </sensor>
     </gazebo>
-    <!-- Diff Drive Plugin (Fortress için uyarlanmış) -->
     <gazebo>
         <plugin
@@ -82,15 +81,13 @@
         </plugin>
         <!-- ROS Kamera Plugin -->
-        <gazebo>
-            <plugin filename="libgazebo_ros_camera.so" name="ros_camera">
-                <ros>
-                    <namespace>/</namespace>
-                </ros>
-                <camera_name>camera</camera_name>
-                <frame_name>camera_optical_link</frame_name>
-                <hack_baseline>0.07</hack_baseline>
-                <update_rate>10</update_rate>
-            </plugin>
-        </gazebo>
+        <plugin filename="libgazebo_ros_camera.so" name="ros_camera">
+            <ros>
+                <namespace>/</namespace>
+            </ros>
+            <camera_name>camera</camera_name>
+            <frame_name>camera_optical_link</frame_name>
+            <hack_baseline>0.07</hack_baseline>
+            <update_rate>10</update_rate>
+        </plugin>
     </gazebo>
 </robot>
