Commit message: robot modelinin boyu küçültüldü. engel kaçışta ufak ayarlamalar yapıldı

File: src/kasva_description/urdf/g_plugins.xacro (robot description, xacro)
@@ -65,13 +65,7 @@
             <topic>cmd_vel</topic>
         </plugin>
-        <plugin filename="libignition-gazebo6-joint-state-publisher-system.so" name="ignition::gazebo::systems::JointStatePublisher">
-            <!-- Yayınlama frekansı (Hz) -->
-            <update_rate>50</update_rate>
-            <!-- Yayınlanacak eklemlerin listesi -->
-            <joint_names>
-                <joint>base_TO_left_wheel</joint>
-                <joint>base_TO_right_wheel</joint>
-                <!-- Diğer eklemleri de ekleyebilirsiniz -->
-            </joint_names>
+        <plugin name="ignition::gazebo::systems::JointStatePublisher" filename="libignition-gazebo-joint-state-publisher-system.so">
+            <update_rate>10</update_rate>
+            <topic>/joint_states</topic>
         </plugin>
         <plugin
@@ -80,4 +74,10 @@
             <render_engine>ogre2</render_engine>
         </plugin>
+        <plugin name="ignition::gazebo::systems::OdometryPublisher" filename="libignition-gazebo-odometry-publisher-system.so">
+            <odom_publish_frequency>10</odom_publish_frequency>
+            <odom_topic>/odom</odom_topic>
+            <odom_frame>odom</odom_frame>
+            <robot_base_frame>base_footprint</robot_base_frame>
+        </plugin>
     </gazebo>
 </robot>

File: src/kasva_description/urdf/rd_props.xacro (robot description, xacro)
@@ -3,5 +3,5 @@
     <!-- l= length, m= mass-->
     <!-- chasis props-->
-    <xacro:property name="chasis_l_x" value="0.6"/>
+    <xacro:property name="chasis_l_x" value="0.4"/>
     <xacro:property name="chasis_l_y" value="0.4"/>
     <xacro:property name="chasis_l_z" value="0.2"/>
@@ -19,4 +19,4 @@
     <xacro:property name="camera_l_y" value="0.1"/>
     <xacro:property name="camera_l_z" value="0.05"/>
-    <xacro:property name="camera_m" value="0.5"/>
+    <xacro:property name="camera_m" value="0.04"/>
 </robot>
